File: harware_design/DrumMachineControlBoard/AnalogIn.sch (KiCad schematic (older format))
At the start: 23 parts, among them J142 Clock_In, J61 AN_IN_AUX_1, J62 AN_IN_AUX_2, J65 AN_IN_AUX_3, J67 AN_IN_AUX_4, J68 AN_IN_AUX_5, Q14 MMBT3904, U14 CD4051B, U15 CD4051B

Commit message: big update, basic drum sequencing is working here
Parts:
- R186, R187: footprint Resistor_SMD:R_0805_2012Metric_Pad1.15x1.40mm_HandSolder -> Resistor_SMD:R_0603_1608Metric_Pad1.05x0.95mm_HandSolder
Changed lines of the file:
@@
 F 0 "R187" V 8545 4750 50  0000 C CNN
 F 1 "10k" V 8636 4750 50  0000 C CNN
-F 2 "Resistor_SMD:R_0805_2012Metric_Pad1.15x1.40mm_HandSolder" V 8790 4740 50  0001 C CNN
+F 2 "Resistor_SMD:R_0603_1608Metric_Pad1.05x0.95mm_HandSolder" V 8790 4740 50  0001 C CNN
 F 3 "~" H 8750 4750 50  0001 C CNN
 	1    8750 4750
@@
 F 0 "R186" H 8182 4254 50  0000 R CNN
 F 1 "10k" H 8182 4345 50  0000 R CNN
-F 2 "Resistor_SMD:R_0805_2012Metric_Pad1.15x1.40mm_HandSolder" V 8290 4290 50  0001 C CNN
+F 2 "Resistor_SMD:R_0603_1608Metric_Pad1.05x0.95mm_HandSolder" V 8290 4290 50  0001 C CNN
 F 3 "~" H 8250 4300 50  0001 C CNN
 	1    8250 4300
