File: harware_design/DrumMachineControlBoard/ButtonInput.sch (KiCad schematic (older format))
At the start: 67 parts, among them SW10 Step8, SW11 inst_sel, SW12 save, SW13 shift, SW14 song, SW15 pattern, SW16 bank, SW17 play/pause, SW18 stop, SW19 Step9, SW20 Step10, SW21 Step11, SW22 Step12, SW23 Step13, SW24 Step14, SW25 Step15, SW26 Step16, SW27 back, SW28 forwards, SW29 mute, SW3 Step1, SW30 step, SW31 beatRep1, SW32 beatRep2, SW4 Step2, SW5 Step3, SW6 Step4, SW7 Step5, SW8 Step6, SW9 Step7, U10 CD4051B, U11 CD4051B, U12 CD4051B, U13 CD4051B, U19 CD4051B

Commit message: big update, basic drum sequencing is working here
Parts:
- R41, R42, R43, R44, R45, R46, R47, R48, R49, R50, R51, R52, R53, R54, R55, R56, R57, R58, R59, R60, R61, R62, R63, R64, R65, R66, R67, R68, R69, R70, R71, R72: footprint Resistor_SMD:R_0805_2012Metric_Pad1.15x1.40mm_HandSolder -> Resistor_SMD:R_0603_1608Metric_Pad1.05x0.95mm_HandSolder
