File: harware_design/DrumMachineControlBoard/Decoupling.sch (KiCad schematic (older format))
At the start: 32 parts

Commit message: big update, basic drum sequencing is working here
Parts:
- added C69, C70: 100n, Capacitor_SMD:C_0603_1608Metric_Pad1.05x0.95mm_HandSolder, symbol Device:C_Small
- C26, C27, C28, C29, C31, C32, C33, C40, C41, C42, C43, C44, C45, C46, C47, C48, C49, C50, C51, C52, C53, C54, C55, C56, C57, C58, C59, C60, C61, C62: footprint Capacitor_SMD:C_0805_2012Metric_Pad1.15x1.40mm_HandSolder -> Capacitor_SMD:C_0603_1608Metric_Pad1.05x0.95mm_HandSolder
- C63, C64: footprint Capacitor_SMD:CP_Elec_4x5.4 -> Capacitor_SMD:CP_Elec_5x5.3
Connections:
- net +12V: now also C69.1, C70.1
- net Earth: now also C69.2, C70.2
