File: harware_design/DrumMachineControlBoard/DrumMachineControlBoard.kicad_pcb (KiCad board)
At the start: 2 copper layers, 385.8 x 170.2 mm, 601 parts, among them J1 TWS_ATT_IN, J10 DIGI3_TRIG_IN, J100 CYNB2-1, J101 Tone2, J102 atk3, J103 CYNB3-1, J104 dist3, J105 snap3w, J106 Tone3, J107 tune3, J108 depth1, J109 dec1w, J11 MIDI IN, J110 tunew, J111 depthw, J112 CYNB4-1, J113 tune1, J114 depth3, J115 dec3, J116 Glitch_LFO, J117 Glitch_In, J118 Kick_Out, J119 Snare_Out, J12 MIDI THRU, J120 CYN1_Out, J121 CYN2_Out, J122 Filt_Aux1, J123 Filt_Aux2, J124 Kick_Vel, J125 Snare_Vel, J126 CYN1_Vel, J127 CYN2_Vel, J128 CYNB5-1, J129 CYNB6-1, J13 MIDI OUT, J130 CYNB1-W3, J131 CYNB2-W3, J132 CYNB3-W3, J133 BD_TRIG_OUT, J134 SN_TRIG_OUT, J135 CYN1_TRIG_OUT, J136 CYN2_TRIG_OUT, J137 GLITCH_TRIG_OUT, J138 DIGI1_TRIG_OUT, J139 DIGI2_TRIG_OUT, J14 BD_Noise, J140 DIGI3_TRIG_OUT, J141 CYNB4-W3, J142 Clock_In, J143 CYNB5-W3, J144 CYNB6-W3, J145 Conn_01x08_Female, J15 Snare_Noise, J16 spk_Conn, J17 out1W, J18 env3, J19 lvl1, J2 Mix_Out, J20 noiseA, J21 DEL_SEND, J22 DEL_REC, J23 Teensy_Audio_OUT_R, J24 freqA, J25 env2, J26 lvl3W, J27 noise/shimA, J28 Teensy_Audio_OUT_L, J29 CYNCM_A, J3 BD_TRIG_IN, J30 HP_A, J31 out3, J32 env1, J33 filter_CV, J34 shimA, J35 BP_A, J36 LP_A, J37 CYNCM_B, J38 res1A, J39 dec1A, J4 SN_TRIG_IN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

Commit message: big update, basic drum sequencing is working here
Parts:
- added C34: 1u, Capacitor_SMD:CP_Elec_4x4.5, B.Cu at (129.5, 24.1)
- added C35: 1u, Capacitor_SMD:CP_Elec_4x4.5, B.Cu at (139.5, 47.0)
- added C38: 10u, Capacitor_SMD:CP_Elec_5x5.3, B.Cu at (112.1, 15.8)
- added C39: 10u, Capacitor_SMD:CP_Elec_5x5.3, B.Cu at (132.1, 37.2)
- added C65: 47n, Capacitor_SMD:C_0603_1608Metric_Pad1.05x0.95mm_HandSolder, B.Cu at (114.0, 21.6)
- added C66: 47n, Capacitor_SMD:C_0603_1608Metric_Pad1.05x0.95mm_HandSolder, B.Cu at (134.4, 42.4)
- added C67: 220u, Capacitor_THT:CP_Radial_D5.0mm_P2.0mm_Bigger_Holes, B.Cu at (112.2, 26.5)
- added C68: 220u, Capacitor_THT:CP_Radial_D5.0mm_P2.0mm_Bigger_Holes, B.Cu at (130.3, 44.7)
- added C69: 100n, Capacitor_SMD:C_0603_1608Metric_Pad1.05x0.95mm_HandSolder, F.Cu at (140.9, 36.5)
- added C70: 100n, Capacitor_SMD:C_0603_1608Metric_Pad1.05x0.95mm_HandSolder, F.Cu at (120.3, 19.0)
- added J146: AuxPot1, Connector_Wire:SolderWirePad_1x01_Drill1mm, F.Cu at (272.4, 42.9)
- added J147: AuxPot2, Connector_Wire:SolderWirePad_1x01_Drill1mm, F.Cu at (277.0, 42.9)
- added J148: AuxPot2, Connector_Wire:SolderWirePad_1x01_Drill1mm, F.Cu at (281.5, 42.9)
- added J149: AuxPot1A, Connector_Wire:SolderWirePad_1x01_Drill1mm, F.Cu at (299.5, 88.9)
- added J150: AuxPot2A, Connector_Wire:SolderWirePad_1x01_Drill1mm, F.Cu at (304.0, 88.9)
- added J151: AuxPot2A, Connector_Wire:SolderWirePad_1x01_Drill1mm, F.Cu at (308.6, 88.9)
- added R183: 470k, Resistor_SMD:R_0603_1608Metric_Pad1.05x0.95mm_HandSolder, B.Cu at (147.2, 8.41)
- added R184: 20k, Resistor_SMD:R_0603_1608Metric_Pad1.05x0.95mm_HandSolder, B.Cu at (147.3, 4.87)
- added R185: 10k, Resistor_SMD:R_0603_1608Metric_Pad1.05x0.95mm_HandSolder, B.Cu at (126.8, 20.4)
- added R201: 10k, Resistor_SMD:R_0603_1608Metric_Pad1.05x0.95mm_HandSolder, B.Cu at (146.9, 38.9)
- added R202: 10, Resistor_SMD:R_0603_1608Metric_Pad1.05x0.95mm_HandSolder, B.Cu at (116.6, 23.8)
- added R203: 10, Resistor_SMD:R_0603_1608Metric_Pad1.05x0.95mm_HandSolder, B.Cu at (135.3, 45.0)
- added R204: 220, Resistor_SMD:R_0603_1608Metric_Pad1.05x0.95mm_HandSolder, B.Cu at (168.6, 10.6)
- added RV54: 100k, mason_parts:masonsPotentiometer_Alpha_RD901F-40-00D_Single_Vertical, F.Cu at (274.4, 39.4)
- added RV55: 100k, mason_parts:masonsPotentiometer_Alpha_RD901F-40-00D_Single_Vertical, F.Cu at (301.4, 85.5)
- added U34: LM386, Package_DIP:DIP-8_W7.62mm_Socket, B.Cu at (144.5, 34.9)
- C1, C10, C11, C12, C13, C14, C16, C18, C19, C2, C20, C21, C22, C23, C25, C26, C27, C28, C29, C3, C31, C32, C33, C36, C4, C40, C41, C42, C43, C44, C45, C46, C47, C48, C49, C50, C51, C52, C53, C54, C55, C56, C57, C58, C59, C60, C61, C62, C9: footprint Capacitor_SMD:C_0805_2012Metric_Pad1.15x1.40mm_HandSolder -> Capacitor_SMD:C_0603_1608Metric_Pad1.05x0.95mm_HandSolder
- C24, C37, C7, C8: footprint Capacitor_SMD:CP_Elec_4x4.5 -> Capacitor_SMD:CP_Elec_5x5.3
- C5: footprint Capacitor_SMD:CP_Elec_6.3x7.7 -> Capacitor_SMD:CP_Elec_8x6.2
- C63, C64: footprint Capacitor_SMD:CP_Elec_4x5.4 -> Capacitor_SMD:CP_Elec_5x5.3
- J11, J12, J13, J145, J74, J79, RV28: moved to B.Cu
- R1, R10, R100, R101, R102, R103, R11, R112, R113, R114, R115, R116, R117, R118, R119, R12, R120, R121, R122, R123, R124, R125, R126, R127, R128, R129, R13, R130, R131, R132, R133, R134, R135, R136, R137, R138, R139, R14, R140, R141, R142, R143, R144, R145, R146, R147, R148, R149, R15, R150, R151, R152, R153, R154, R155, R156, R157, R158, R159, R16, R160, R161, R162, R163, R164, R165, R166, R167, R168, R169, R17, R170, R171, R172, R173, R174, R177, R178, R179, R18, R180, R186, R187, R19, R194, R195, R196, R197, R198, R2, R20, R206, R21, R22, R23, R24, R25, R26, R27, R28, R29, R3, R30, R31, R32, R33, R34, R35, R36, R37, R38, R39, R4, R40, R41, R42, R43, R44, R45, R46, R47, R48, R49, R5, R50, R51, R52, R53, R54, R55, R56, R57, R58, R59, R6, R60, R61, R62, R63, R64, R65, R66, R67, R68, R69, R7, R70, R71, R72, R73, R74, R75, R76, R77, R78, R79, R8, R80, R81, R82, R83, R84, R85, R86, R87, R88, R89, R9, R90, R91, R92, R93, R94, R95, R96, R97, R98, R99: footprint Resistor_SMD:R_0805_2012Metric_Pad1.15x1.40mm_HandSolder -> Resistor_SMD:R_0603_1608Metric_Pad1.05x0.95mm_HandSolder
- R104, R105, R106, R107, R108, R109, R110, R111, R175, R176, R181, R182, R188, R189, R190, R191, R192, R193, R207, R208: footprint Capacitor_SMD:C_0805_2012Metric_Pad1.15x1.40mm_HandSolder -> Resistor_SMD:R_0603_1608Metric_Pad1.05x0.95mm_HandSolder
- RV53: value 10k -> 100k; footprint Potentiometer_THT:Potentiometer_Runtron_RM-065_Vertical -> mason_parts:masonsPotentiometer_Alpha_RD901F-40-00D_Single_Vertical
- RV59: footprint mason_parts:masonsPotentiometer_Alpha_RD901F-40-00D_Single_Vertical -> mason_parts:Amphenol_Trimpot
- U33: value TL072 -> LM386; footprint Package_SO:SOIC-8_3.9x4.9mm_P1.27mm -> Package_DIP:DIP-8_W7.62mm_Socket
- moved RV53 20.4 mm to (134.4, 11.5), turned to 90 degrees
- moved U33 9.61 mm to (124.4, 13.7), turned to 180 degrees
- moved D6 8.20 mm to (368.4, 81.6), turned to 190 degrees
- moved RV28 7.25 mm to (375.4, 39.5), turned to 0 degrees
- moved C7 4.15 mm to (373.8, 77.5), turned to 30 degrees
- moved C5 2.40 mm to (357.5, 73.0)
- moved J79 1.73 mm to (271.0, 3.35)
- moved RV23 0.81 mm to (259.5, 91.0)
- moved J74 0.81 mm to (258.9, 9.69)
- moved C24 0.53 mm to (394.5, 23.8)
- moved C64 0.43 mm to (192.0, 77.1)
- moved RV59 0.40 mm to (34.0, 30.9), turned to 0 degrees
- moved JP1 0.30 mm to (259.0, 73.9)
- moved J11 0.19 mm to (182.6, 7.49)
- moved J12 0.16 mm to (206.2, 7.46)
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Connections:
- net MEM_MISO renamed Net-(U5-Pad14)
- J76 pad R1: Net-(J76-PadR1) -> Net-(C68-Pad2)
- J76 pad T1: Net-(J76-PadT1) -> Net-(C67-Pad2)
- RV53 pad 1: Earth -> LINE_OUT
- RV53 pad 2: Net-(RV53-Pad2) -> Net-(R183-Pad2)
- RV53 pad 3: LINE_OUT -> Earth
- U33 pad 1: Net-(J76-PadR1) -> Net-(U33-Pad1)
- U33 pad 2: Net-(J76-PadR1) -> Earth
- U33 pad 3: Net-(RV53-Pad2) -> Net-(C34-Pad1)
- U33 pad 4: -12V -> Earth
- U33 pad 5: Net-(RV53-Pad2) -> Net-(C65-Pad1)
- U33 pad 6: Net-(J76-PadT1) -> +12V
- U33 pad 7: Net-(J76-PadT1) -> Net-(C38-Pad1)
- U33 pad 8: +12V -> Net-(U33-Pad8)
- U5 pad 13: MEM_MOSI -> Net-(U5-Pad13)
Routing:
- net -12V: track 1074.4 -> 787.0 mm, vias 17 -> 15
- net Earth: track 3484.6 -> 3621.0 mm, vias 47 -> 46
- net Net-(C68-Pad2): track 0.00 -> 65.1 mm, vias 0 -> 1
- net Net-(C34-Pad2): track 0.00 -> 61.4 mm, vias 0 -> 2
- net Net-(C67-Pad2): track 0.00 -> 58.7 mm, vias 0 -> 1
- net Net-(J12-Pad4): track 0.00 -> 53.0 mm
- net Net-(J76-PadR1): track 48.9 -> 0.00 mm
- net Net-(J76-PadT1): track 40.7 -> 0.00 mm
- net +12V: track 1326.6 -> 1352.2 mm
- net Net-(J11-Pad4): track 11.4 -> 34.8 mm
- net Net-(RV53-Pad2): track 22.4 -> 0.00 mm, vias 2 -> 0
- net Net-(J92-Pad1): track 5.63 -> 22.2 mm
- net +5V: track 850.5 -> 865.8 mm
- net Net-(J13-Pad4): track 34.0 -> 48.3 mm
- net LINE_OUT: track 347.7 -> 334.9 mm, vias 1 -> 0
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Other:
- board text added: "POWER IN"
- board text added: "TO POWER BOARD"
