File: harware_design/DrumMachineControlBoard/DrumMachineControlBoard.sch (KiCad schematic (older format))
At the start: 6 parts, among them J23 Teensy_Audio_OUT_R, J28 Teensy_Audio_OUT_L, J46 Clock_Out, J54 Teensy_27, U25 Teensy_Audio_Shield, U5 Teensy4.1

Commit message: big update, basic drum sequencing is working here
Connections:
- net MEM_MISO: no longer U5.14 (12_MISO_MQSL)
- net MEM_MOSI: no longer U5.13 (11_MOSI_CTX1)
- no-connect marks 81 -> 73
Changed lines of the file:
@@
 Text GLabel 1850 1750 0    50   BiDi ~ 0
 MEM_CS
-Text GLabel 1850 2250 0    50   BiDi ~ 0
+Text GLabel 1800 2250 0    50   BiDi ~ 0
 MEM_MOSI
 Text GLabel 4050 2350 2    50   BiDi ~ 0
@@
 Text GLabel 1850 2150 0    50   BiDi ~ 0
 LCD_CS
-Text GLabel 950  2750 0    50   BiDi ~ 0
-LCD_MOSI
-Text GLabel 950  2850 0    50   BiDi ~ 0
-LCD_SCK
 Text GLabel 1850 3350 0    50   BiDi ~ 0
 LED_LATCH
@@
 Text GLabel 1850 2650 0    50   BiDi ~ 0
 LCD_DC
-Text GLabel 1850 2350 0    50   BiDi ~ 0
+Text GLabel 1800 2350 0    50   BiDi ~ 0
 MEM_MISO
-$Comp
-L power:Earth #PWR0221
-U 1 1 63208D90
-P 2350 5100
-F 0 "#PWR0221" H 2350 4850 50  0001 C CNN
-F 1 "Earth" H 2350 4950 50  0001 C CNN
-F 2 "" H 2350 5100 50  0001 C CNN
-F 3 "~" H 2350 5100 50  0001 C CNN
-	1    2350 5100
+Text GLabel 5100 7200 2    50   BiDi ~ 0
+D_Aud_R
+Text GLabel 5100 7400 2    50   BiDi ~ 0
+D_Aud_L
+$Comp
+L teensy:Teensy4.1 U5
+U 1 1 630E849F
+P 2950 3200
+F 0 "U5" H 2950 5765 50  0000 C CNN
+F 1 "Teensy4.1" H 2950 5674 50  0000 C CNN
+F 2 "teensy pretty:Teensy41" H 2550 3600 50  0001 C CNN
+F 3 "" H 2550 3600 50  0001 C CNN
+	1    2950 3200
+	1    0    0    -1
+$EndComp
+$Comp
+L power:+3.3V #PWR025
+U 1 1 632B6240
+P 4050 1250
+F 0 "#PWR025" H 4050 1100 50  0001 C CNN
+F 1 "+3.3V" V 4065 1378 50  0000 L CNN
+F 2 "" H 4050 1250 50  0001 C CNN
+F 3 "" H 4050 1250 50  0001 C CNN
+	1    4050 1250
 	0    1    1    0
 $EndComp
+$Sheet
+S 9400 2900 550  300
+U 6341C53F
+F0 "Noise" 50
+F1 "Noise.sch" 50
+$EndSheet
+Text GLabel 4050 3050 2    50   BiDi ~ 0
+CLOCK_IN
+$Comp
+L Connector:Conn_01x01_Female J?
+U 1 1 636D367B
+P 1650 2750
+AR Path="/6303B621/636D367B" Ref="J?"  Part="1"
+AR Path="/636D367B" Ref="J46"  Part="1"
+F 0 "J46" H 1678 2776 50  0000 L CNN
+F 1 "Clock_Out" H 1800 2750 50  0000 L CNN
+F 2 "Connector_Wire:SolderWirePad_1x01_Drill1mm" H 1650 2750 50  0001 C CNN
+F 3 "~" H 1650 2750 50  0001 C CNN
+	1    1650 2750
+	-1   0    0    1
+$EndComp
+$Sheet
+S 9400 3450 550  300
+U 6370FEA3
+F0 "power_conns" 50
+F1 "power_conns.sch" 50
+$EndSheet
+$Sheet
+S 9400 3950 550  350
+U 6346700D
+F0 "SpeakerAmp" 50
+F1 "SpeakerAmp.sch" 50
+$EndSheet
+$Sheet
+S 9400 2350 550  300
+U 630FA783
+F0 "PWM Out" 50
+F1 "PWM Out.sch" 50
+$EndSheet
+$Comp
+L Connector:Conn_01x01_Female J28
+U 1 1 635C6C6F
+P 4900 7400
+F 0 "J28" H 4928 7426 50  0000 L CNN
+F 1 "Teensy_Audio_OUT_L" H 4928 7335 50  0000 L CNN
+F 2 "Connector_Wire:SolderWirePad_1x01_Drill1mm" H 4900 7400 50  0001 C CNN
+F 3 "~" H 4900 7400 50  0001 C CNN
+	1    4900 7400
+	-1   0    0    1
+$EndComp
+$Comp
+L Connector:Conn_01x01_Female J23
+U 1 1 635C6FCF
+P 4900 7200
+F 0 "J23" H 4928 7226 50  0000 L CNN
+F 1 "Teensy_Audio_OUT_R" H 4928 7135 50  0000 L CNN
+F 2 "Connector_Wire:SolderWirePad_1x01_Drill1mm" H 4900 7200 50  0001 C CNN
+F 3 "~" H 4900 7200 50  0001 C CNN
+	1    4900 7200
+	-1   0    0    1
+$EndComp
+$Comp
+L Connector:Conn_01x01_Female J54
+U 1 1 636C4AD8
+P 1650 2850
+F 0 "J54" H 2100 2850 50  0000 C CNN
+F 1 "Teensy_27" H 1850 2850 50  0000 C CNN
+F 2 "Connector_Wire:SolderWirePad_1x01_Drill1mm" H 1650 2850 50  0001 C CNN
+F 3 "~" H 1650 2850 50  0001 C CNN
+	1    1650 2850
+	-1   0    0    1
+$EndComp
+$Sheet
+S 9400 4500 550  350
+U 6372203A
+F0 "Decoupling" 50
+F1 "Decoupling.sch" 50
+$EndSheet
+$Sheet
+S 9400 5100 550  300
+U 63A851CD
+F0 "JackPanel" 50
+F1 "JackPanel.sch" 50
+$EndSheet
 NoConn ~ 3450 5500
 Text GLabel 2300 5800 0    50   BiDi ~ 0
 MEM_CS
-Text GLabel 2300 6300 0    50   BiDi ~ 0
-MEM_MOSI
-Text GLabel 2300 6400 0    50   BiDi ~ 0
-MEM_MISO
 Text GLabel 3600 6400 2    50   BiDi ~ 0
 MEM_SCK
@@
 NoConn ~ 3450 7500
 NoConn ~ 3450 7300
-Text GLabel 5100 7200 2    50   BiDi ~ 0
-D_Aud_R
-Text GLabel 5100 7400 2    50   BiDi ~ 0
-D_Aud_L
 NoConn ~ 3100 4850
 NoConn ~ 2900 4850
-$Comp
-L teensy:Teensy4.1 U5
-U 1 1 630E849F
-P 2950 3200
-F 0 "U5" H 2950 5765 50  0000 C CNN
-F 1 "Teensy4.1" H 2950 5674 50  0000 C CNN
-F 2 "teensy pretty:Teensy41" H 2550 3600 50  0001 C CNN
-F 3 "" H 2550 3600 50  0001 C CNN
-	1    2950 3200
-	1    0    0    -1
-$EndComp
-$Comp
-L power:+3.3V #PWR025
-U 1 1 632B6240
-P 4050 1250
-F 0 "#PWR025" H 4050 1100 50  0001 C CNN
-F 1 "+3.3V" V 4065 1378 50  0000 L CNN
-F 2 "" H 4050 1250 50  0001 C CNN
-F 3 "" H 4050 1250 50  0001 C CNN
-	1    4050 1250
-	0    1    1    0
-$EndComp
-$Sheet
-S 9400 2900 550  300
-U 6341C53F
-F0 "Noise" 50
-F1 "Noise.sch" 50
-$EndSheet
-Text GLabel 4050 3050 2    50   BiDi ~ 0
-CLOCK_IN
-$Comp
-L Connector:Conn_01x01_Female J?
-U 1 1 636D367B
-P 1650 2750
-AR Path="/6303B621/636D367B" Ref="J?"  Part="1"
-AR Path="/636D367B" Ref="J46"  Part="1"
-F 0 "J46" H 1678 2776 50  0000 L CNN
-F 1 "Clock_Out" H 1800 2750 50  0000 L CNN
-F 2 "Connector_Wire:SolderWirePad_1x01_Drill1mm" H 1650 2750 50  0001 C CNN
-F 3 "~" H 1650 2750 50  0001 C CNN
-	1    1650 2750
-	-1   0    0    1
-$EndComp
-NoConn ~ 950  2750
-NoConn ~ 950  2850
-$Sheet
-S 9400 3450 550  300
-U 6370FEA3
-F0 "power_conns" 50
-F1 "power_conns.sch" 50
-$EndSheet
-$Sheet
-S 9400 3950 550  350
-U 6346700D
-F0 "SpeakerAmp" 50
-F1 "SpeakerAmp.sch" 50
-$EndSheet
-$Sheet
-S 9400 2350 550  300
-U 630FA783
-F0 "PWM Out" 50
-F1 "PWM Out.sch" 50
-$EndSheet
-$Comp
-L Connector:Conn_01x01_Female J28
-U 1 1 635C6C6F
-P 4900 7400
-F 0 "J28" H 4928 7426 50  0000 L CNN
-F 1 "Teensy_Audio_OUT_L" H 4928 7335 50  0000 L CNN
-F 2 "Connector_Wire:SolderWirePad_1x01_Drill1mm" H 4900 7400 50  0001 C CNN
-F 3 "~" H 4900 7400 50  0001 C CNN
-	1    4900 7400
-	-1   0    0    1
-$EndComp
-$Comp
-L Connector:Conn_01x01_Female J23
-U 1 1 635C6FCF
-P 4900 7200
-F 0 "J23" H 4928 7226 50  0000 L CNN
-F 1 "Teensy_Audio_OUT_R" H 4928 7135 50  0000 L CNN
-F 2 "Connector_Wire:SolderWirePad_1x01_Drill1mm" H 4900 7200 50  0001 C CNN
-F 3 "~" H 4900 7200 50  0001 C CNN
-	1    4900 7200
-	-1   0    0    1
-$EndComp
 NoConn ~ 3450 6700
 NoConn ~ 3450 6800
@@
 NoConn ~ 2300 5900
 NoConn ~ 2300 6000
-NoConn ~ 2300 6300
-NoConn ~ 2300 6400
 NoConn ~ 2450 6400
 NoConn ~ 2450 6300
@@
 NoConn ~ 2450 5900
 NoConn ~ 2450 5100
-NoConn ~ 2350 5100
-$Comp
-L power:+5V #PWR024
-U 1 1 632B3794
-P 3600 5100
-F 0 "#PWR024" H 3600 4950 50  0001 C CNN
-F 1 "+5V" V 3615 5228 50  0000 L CNN
-F 2 "" H 3600 5100 50  0001 C CNN
-F 3 "" H 3600 5100 50  0001 C CNN
-	1    3600 5100
-	0    1    1    0
-$EndComp
 Text GLabel 3600 5900 2    50   BiDi ~ 0
 AUD_SDA
@@
 Text GLabel 3600 5400 2    50   BiDi ~ 0
 AUD_MCLK
-$Comp
-L power:+3.3V #PWR0222
-U 1 1 6320BBAF
-P 3600 5300
-F 0 "#PWR0222" H 3600 5150 50  0001 C CNN
-F 1 "+3.3V" V 3615 5428 50  0000 L CNN
-F 2 "" H 3600 5300 50  0001 C CNN
-F 3 "" H 3600 5300 50  0001 C CNN
-	1    3600 5300
-	0    1    1    0
-$EndComp
-$Comp
-L power:Earth #PWR0220
-U 1 1 6320854A
-P 3600 5200
-F 0 "#PWR0220" H 3600 4950 50  0001 C CNN
-F 1 "Earth" H 3600 5050 50  0001 C CNN
-F 2 "" H 3600 5200 50  0001 C CNN
-F 3 "~" H 3600 5200 50  0001 C CNN
-	1    3600 5200
-	0    -1   -1   0
-$EndComp
+NoConn ~ 3450 5100
+NoConn ~ 3450 5200
+NoConn ~ 3450 5300
+NoConn ~ 3450 5400
+NoConn ~ 3450 5600
+NoConn ~ 3450 5700
+NoConn ~ 3450 5800
+NoConn ~ 3450 5900
+NoConn ~ 3600 5400
+NoConn ~ 3600 5600
+NoConn ~ 3600 5700
+NoConn ~ 3600 5800
+NoConn ~ 3600 5900
+NoConn ~ 3450 6400
 $Comp
 L modular_synth:Teensy_Audio_Shield U25
@@
 	1    0    0    -1
 $EndComp
-NoConn ~ 3850 5200
-NoConn ~ 3450 5100
-NoConn ~ 3450 5200
-NoConn ~ 3450 5300
-NoConn ~ 3450 5400
-NoConn ~ 3450 5600
-NoConn ~ 3450 5700
-NoConn ~ 3450 5800
-NoConn ~ 3450 5900
-NoConn ~ 3600 5100
-NoConn ~ 3600 5200
-NoConn ~ 3600 5300
-NoConn ~ 3600 5400
-NoConn ~ 3600 5600
-NoConn ~ 3600 5700
-NoConn ~ 3600 5800
-NoConn ~ 3600 5900
-NoConn ~ 3450 6400
-NoConn ~ 3600 6400
-$Comp
-L Connector:Conn_01x01_Female J54
-U 1 1 636C4AD8
-P 1650 2850
-F 0 "J54" H 2100 2850 50  0000 C CNN
-F 1 "Teensy_27" H 1850 2850 50  0000 C CNN
-F 2 "Connector_Wire:SolderWirePad_1x01_Drill1mm" H 1650 2850 50  0001 C CNN
-F 3 "~" H 1650 2850 50  0001 C CNN
-	1    1650 2850
-	-1   0    0    1
-$EndComp
-$Sheet
-S 9400 4500 550  350
-U 6372203A
-F0 "Decoupling" 50
-F1 "Decoupling.sch" 50
-$EndSheet
-$Sheet
-S 9400 5100 550  300
-U 63A851CD
-F0 "JackPanel" 50
-F1 "JackPanel.sch" 50
-$EndSheet
+Text GLabel 2300 6300 0    50   BiDi ~ 0
+MEM_MOSI
+Text GLabel 2300 6400 0    50   BiDi ~ 0
+MEM_MISO
+NoConn ~ 1850 2250
+NoConn ~ 1850 2350
 $EndSCHEMATC
