File: harware_design/DrumMachineControlBoard/ExternalPots.sch (KiCad schematic (older format))
At the start: 74 parts, among them J101 Tone2, J102 atk3, J104 dist3, J105 snap3w, J106 Tone3, J107 tune3, J108 depth1, J109 dec1w, J110 tunew, J111 depthw, J113 tune1, J114 depth3, J115 dec3, J17 out1W, J18 env3, J19 lvl1, J20 noiseA, J24 freqA, J25 env2, J26 lvl3W, J27 noise/shimA, J29 CYNCM_A, J30 HP_A, J31 out3, J32 env1, J34 shimA, J35 BP_A, J36 LP_A, J37 CYNCM_B, J38 res1A, J39 dec1A, J41 HP_B, J42 BP_B, J43 LP_B, J44 res23A, J45 dec23A, J57 Env_1B, J59 noiseB, J63 freqB, J64 Env_2B, J66 noise/shimB, J71 Env_3B, J73 shimB, J77 res1B, J78 dec1B, J83 res23B, J84 dec23B, J92 atk1W, J93 tune, J94 dist1W, J95 snap1, J96 Tone1, U26 SP3TCYNA, U27 SP3TCYNB

Commit message: big update, basic drum sequencing is working here
Parts:
- added J146: AuxPot1, Connector_Wire:SolderWirePad_1x01_Drill1mm, symbol Connector:Conn_01x01_Female
- added J147, J148: AuxPot2, Connector_Wire:SolderWirePad_1x01_Drill1mm, symbol Connector:Conn_01x01_Female
- added J149: AuxPot1A, Connector_Wire:SolderWirePad_1x01_Drill1mm, symbol Connector:Conn_01x01_Female
- added J150, J151: AuxPot2A, Connector_Wire:SolderWirePad_1x01_Drill1mm, symbol Connector:Conn_01x01_Female
- added RV54, RV55: 100k, mason_parts:masonsPotentiometer_Alpha_RD901F-40-00D_Single_Vertical, symbol Device:R_POT_US
- RV59: footprint mason_parts:masonsPotentiometer_Alpha_RD901F-40-00D_Single_Vertical -> mason_parts:Amphenol_Trimpot
Connections:
- new net: J146.1 (Pin_1), RV54.1
- new net: J147.1 (Pin_1), RV54.2
- new net: J148.1 (Pin_1), RV54.3
- new net: J149.1 (Pin_1), RV55.1
- new net: J150.1 (Pin_1), RV55.2
- new net: J151.1 (Pin_1), RV55.3
Changed lines of the file:
@@
 F 0 "RV59" V 5987 1250 50  0000 C CNN
 F 1 "470" V 5896 1250 50  0000 C CNN
-F 2 "mason_parts:masonsPotentiometer_Alpha_RD901F-40-00D_Single_Vertical" H 6100 1250 50  0001 C CNN
+F 2 "mason_parts:Amphenol_Trimpot" H 6100 1250 50  0001 C CNN
 F 3 "~" H 6100 1250 50  0001 C CNN
 	1    6100 1250
@@
 	5950 2450 5900 2450
 Connection ~ 5950 2450
+$Comp
+L Device:R_POT_US RV54
+U 1 1 6381F021
+P 2250 6700
+F 0 "RV54" V 2137 6700 50  0000 C CNN
+F 1 "100k" V 2046 6700 50  0000 C CNN
+F 2 "mason_parts:masonsPotentiometer_Alpha_RD901F-40-00D_Single_Vertical" H 2250 6700 50  0001 C CNN
+F 3 "~" H 2250 6700 50  0001 C CNN
+	1    2250 6700
+	0    -1   -1   0
+$EndComp
+$Comp
+L Connector:Conn_01x01_Female J148
+U 1 1 6381F027
+P 2600 6700
+F 0 "J148" H 2628 6726 50  0000 L CNN
+F 1 "AuxPot2" H 2450 6650 50  0000 L CNN
+F 2 "Connector_Wire:SolderWirePad_1x01_Drill1mm" H 2600 6700 50  0001 C CNN
+F 3 "~" H 2600 6700 50  0001 C CNN
+	1    2600 6700
+	1    0    0    -1
+$EndComp
+$Comp
+L Connector:Conn_01x01_Female J147
+U 1 1 6381F02D
+P 2250 6350
+F 0 "J147" V 2188 6262 50  0000 R CNN
+F 1 "AuxPot2" V 2097 6262 50  0000 R CNN
+F 2 "Connector_Wire:SolderWirePad_1x01_Drill1mm" H 2250 6350 50  0001 C CNN
+F 3 "~" H 2250 6350 50  0001 C CNN
+	1    2250 6350
+	0    -1   -1   0
+$EndComp
+$Comp
+L Connector:Conn_01x01_Female J146
+U 1 1 6381F033
+P 1900 6700
+F 0 "J146" H 1792 6475 50  0000 C CNN
+F 1 "AuxPot1" H 1792 6566 50  0000 C CNN
+F 2 "Connector_Wire:SolderWirePad_1x01_Drill1mm" H 1900 6700 50  0001 C CNN
+F 3 "~" H 1900 6700 50  0001 C CNN
+	1    1900 6700
+	-1   0    0    1
+$EndComp
+$Comp
+L Device:R_POT_US RV55
+U 1 1 638202BE
+P 3350 6700
+F 0 "RV55" V 3237 6700 50  0000 C CNN
+F 1 "100k" V 3146 6700 50  0000 C CNN
+F 2 "mason_parts:masonsPotentiometer_Alpha_RD901F-40-00D_Single_Vertical" H 3350 6700 50  0001 C CNN
+F 3 "~" H 3350 6700 50  0001 C CNN
+	1    3350 6700
+	0    -1   -1   0
+$EndComp
+$Comp
+L Connector:Conn_01x01_Female J151
+U 1 1 638202C4
+P 3700 6700
+F 0 "J151" H 3728 6726 50  0000 L CNN
+F 1 "AuxPot2A" H 3550 6650 50  0000 L CNN
+F 2 "Connector_Wire:SolderWirePad_1x01_Drill1mm" H 3700 6700 50  0001 C CNN
+F 3 "~" H 3700 6700 50  0001 C CNN
+	1    3700 6700
+	1    0    0    -1
+$EndComp
+$Comp
+L Connector:Conn_01x01_Female J150
+U 1 1 638202CA
+P 3350 6350
+F 0 "J150" V 3288 6262 50  0000 R CNN
+F 1 "AuxPot2A" V 3197 6262 50  0000 R CNN
+F 2 "Connector_Wire:SolderWirePad_1x01_Drill1mm" H 3350 6350 50  0001 C CNN
+F 3 "~" H 3350 6350 50  0001 C CNN
+	1    3350 6350
+	0    -1   -1   0
+$EndComp
+$Comp
+L Connector:Conn_01x01_Female J149
+U 1 1 638202D0
+P 3000 6700
+F 0 "J149" H 2892 6475 50  0000 C CNN
+F 1 "AuxPot1A" H 2892 6566 50  0000 C CNN
+F 2 "Connector_Wire:SolderWirePad_1x01_Drill1mm" H 3000 6700 50  0001 C CNN
+F 3 "~" H 3000 6700 50  0001 C CNN
+	1    3000 6700
+	-1   0    0    1
+$EndComp
 $EndSCHEMATC
