File: harware_design/DrumMachineControlBoard/ExternalTrigger.sch (KiCad schematic (older format))
At the start: 40 parts, among them J10 DIGI3_TRIG_IN, J3 BD_TRIG_IN, J4 SN_TRIG_IN, J5 CYN1_TRIG_IN, J6 CYN2_TRIG_IN, J7 GLITCH_TRIG_IN, J8 DIGI1_TRIG_IN, J9 DIGI2_TRIG_IN, Q10 MMBT3904, Q3 MMBT3904, Q4 MMBT3904, Q5 MMBT3904, Q6 MMBT3904, Q7 MMBT3904, Q8 MMBT3904, Q9 MMBT3904

Commit message: big update, basic drum sequencing is working here
Parts:
- R112, R113, R114, R115, R116, R117, R118, R119, R120, R121, R122, R123, R124, R125, R126, R127: footprint Resistor_SMD:R_0805_2012Metric_Pad1.15x1.40mm_HandSolder -> Resistor_SMD:R_0603_1608Metric_Pad1.05x0.95mm_HandSolder
Changed lines of the file:
@@
 F 0 "R112" V 995 1750 50  0000 C CNN
 F 1 "10k" V 1086 1750 50  0000 C CNN
-F 2 "Resistor_SMD:R_0805_2012Metric_Pad1.15x1.40mm_HandSolder" V 1240 1740 50  0001 C CNN
+F 2 "Resistor_SMD:R_0603_1608Metric_Pad1.05x0.95mm_HandSolder" V 1240 1740 50  0001 C CNN
 F 3 "~" H 1200 1750 50  0001 C CNN
 	1    1200 1750
@@
 F 0 "R116" H 1632 1254 50  0000 R CNN
 F 1 "10k" H 1632 1345 50  0000 R CNN
-F 2 "Resistor_SMD:R_0805_2012Metric_Pad1.15x1.40mm_HandSolder" V 1740 1290 50  0001 C CNN
+F 2 "Resistor_SMD:R_0603_1608Metric_Pad1.05x0.95mm_HandSolder" V 1740 1290 50  0001 C CNN
 F 3 "~" H 1700 1300 50  0001 C CNN
 	1    1700 1300
@@
 F 0 "R113" V 995 2900 50  0000 C CNN
 F 1 "10k" V 1086 2900 50  0000 C CNN
-F 2 "Resistor_SMD:R_0805_2012Metric_Pad1.15x1.40mm_HandSolder" V 1240 2890 50  0001 C CNN
+F 2 "Resistor_SMD:R_0603_1608Metric_Pad1.05x0.95mm_HandSolder" V 1240 2890 50  0001 C CNN
 F 3 "~" H 1200 2900 50  0001 C CNN
 	1    1200 2900
@@
 F 0 "R117" H 1632 2404 50  0000 R CNN
 F 1 "10k" H 1632 2495 50  0000 R CNN
-F 2 "Resistor_SMD:R_0805_2012Metric_Pad1.15x1.40mm_HandSolder" V 1740 2440 50  0001 C CNN
+F 2 "Resistor_SMD:R_0603_1608Metric_Pad1.05x0.95mm_HandSolder" V 1740 2440 50  0001 C CNN
 F 3 "~" H 1700 2450 50  0001 C CNN
 	1    1700 2450
@@
 F 0 "R114" V 995 4050 50  0000 C CNN
 F 1 "10k" V 1086 4050 50  0000 C CNN
-F 2 "Resistor_SMD:R_0805_2012Metric_Pad1.15x1.40mm_HandSolder" V 1240 4040 50  0001 C CNN
+F 2 "Resistor_SMD:R_0603_1608Metric_Pad1.05x0.95mm_HandSolder" V 1240 4040 50  0001 C CNN
 F 3 "~" H 1200 4050 50  0001 C CNN
 	1    1200 4050
@@
 F 0 "R118" H 1632 3554 50  0000 R CNN
 F 1 "10k" H 1632 3645 50  0000 R CNN
-F 2 "Resistor_SMD:R_0805_2012Metric_Pad1.15x1.40mm_HandSolder" V 1740 3590 50  0001 C CNN
+F 2 "Resistor_SMD:R_0603_1608Metric_Pad1.05x0.95mm_HandSolder" V 1740 3590 50  0001 C CNN
 F 3 "~" H 1700 3600 50  0001 C CNN
 	1    1700 3600
@@
 F 0 "R115" V 995 5200 50  0000 C CNN
 F 1 "10k" V 1086 5200 50  0000 C CNN
-F 2 "Resistor_SMD:R_0805_2012Metric_Pad1.15x1.40mm_HandSolder" V 1240 5190 50  0001 C CNN
+F 2 "Resistor_SMD:R_0603_1608Metric_Pad1.05x0.95mm_HandSolder" V 1240 5190 50  0001 C CNN
 F 3 "~" H 1200 5200 50  0001 C CNN
 	1    1200 5200
@@
 F 0 "R119" H 1632 4704 50  0000 R CNN
 F 1 "10k" H 1632 4795 50  0000 R CNN
-F 2 "Resistor_SMD:R_0805_2012Metric_Pad1.15x1.40mm_HandSolder" V 1740 4740 50  0001 C CNN
+F 2 "Resistor_SMD:R_0603_1608Metric_Pad1.05x0.95mm_HandSolder" V 1740 4740 50  0001 C CNN
 F 3 "~" H 1700 4750 50  0001 C CNN
 	1    1700 4750
@@
 F 0 "R120" V 2495 1750 50  0000 C CNN
 F 1 "10k" V 2586 1750 50  0000 C CNN
-F 2 "Resistor_SMD:R_0805_2012Metric_Pad1.15x1.40mm_HandSolder" V 2740 1740 50  0001 C CNN
+F 2 "Resistor_SMD:R_0603_1608Metric_Pad1.05x0.95mm_HandSolder" V 2740 1740 50  0001 C CNN
 F 3 "~" H 2700 1750 50  0001 C CNN
 	1    2700 1750
@@
 F 0 "R124" H 3132 1254 50  0000 R CNN
 F 1 "10k" H 3132 1345 50  0000 R CNN
-F 2 "Resistor_SMD:R_0805_2012Metric_Pad1.15x1.40mm_HandSolder" V 3240 1290 50  0001 C CNN
+F 2 "Resistor_SMD:R_0603_1608Metric_Pad1.05x0.95mm_HandSolder" V 3240 1290 50  0001 C CNN
 F 3 "~" H 3200 1300 50  0001 C CNN
 	1    3200 1300
@@
 F 0 "R121" V 2495 2900 50  0000 C CNN
 F 1 "10k" V 2586 2900 50  0000 C CNN
-F 2 "Resistor_SMD:R_0805_2012Metric_Pad1.15x1.40mm_HandSolder" V 2740 2890 50  0001 C CNN
+F 2 "Resistor_SMD:R_0603_1608Metric_Pad1.05x0.95mm_HandSolder" V 2740 2890 50  0001 C CNN
 F 3 "~" H 2700 2900 50  0001 C CNN
 	1    2700 2900
@@
 F 0 "R125" H 3132 2404 50  0000 R CNN
 F 1 "10k" H 3132 2495 50  0000 R CNN
-F 2 "Resistor_SMD:R_0805_2012Metric_Pad1.15x1.40mm_HandSolder" V 3240 2440 50  0001 C CNN
+F 2 "Resistor_SMD:R_0603_1608Metric_Pad1.05x0.95mm_HandSolder" V 3240 2440 50  0001 C CNN
 F 3 "~" H 3200 2450 50  0001 C CNN
 	1    3200 2450
@@
 F 0 "R122" V 2495 4050 50  0000 C CNN
 F 1 "10k" V 2586 4050 50  0000 C CNN
-F 2 "Resistor_SMD:R_0805_2012Metric_Pad1.15x1.40mm_HandSolder" V 2740 4040 50  0001 C CNN
+F 2 "Resistor_SMD:R_0603_1608Metric_Pad1.05x0.95mm_HandSolder" V 2740 4040 50  0001 C CNN
 F 3 "~" H 2700 4050 50  0001 C CNN
 	1    2700 4050
@@
 F 0 "R126" H 3132 3554 50  0000 R CNN
 F 1 "10k" H 3132 3645 50  0000 R CNN
-F 2 "Resistor_SMD:R_0805_2012Metric_Pad1.15x1.40mm_HandSolder" V 3240 3590 50  0001 C CNN
+F 2 "Resistor_SMD:R_0603_1608Metric_Pad1.05x0.95mm_HandSolder" V 3240 3590 50  0001 C CNN
 F 3 "~" H 3200 3600 50  0001 C CNN
 	1    3200 3600
@@
 F 0 "R123" V 2495 5200 50  0000 C CNN
 F 1 "10k" V 2586 5200 50  0000 C CNN
-F 2 "Resistor_SMD:R_0805_2012Metric_Pad1.15x1.40mm_HandSolder" V 2740 5190 50  0001 C CNN
+F 2 "Resistor_SMD:R_0603_1608Metric_Pad1.05x0.95mm_HandSolder" V 2740 5190 50  0001 C CNN
 F 3 "~" H 2700 5200 50  0001 C CNN
 	1    2700 5200
@@
 F 0 "R127" H 3132 4704 50  0000 R CNN
 F 1 "10k" H 3132 4795 50  0000 R CNN
-F 2 "Resistor_SMD:R_0805_2012Metric_Pad1.15x1.40mm_HandSolder" V 3240 4740 50  0001 C CNN
+F 2 "Resistor_SMD:R_0603_1608Metric_Pad1.05x0.95mm_HandSolder" V 3240 4740 50  0001 C CNN
 F 3 "~" H 3200 4750 50  0001 C CNN
 	1    3200 4750
