File: harware_design/DrumMachineControlBoard/GlitchVoice.sch (KiCad schematic (older format))
At the start: 61 parts, among them J1 TWS_ATT_IN, J116 Glitch_LFO, J117 Glitch_In, J72 TWS_ATT_OUT, Q11 MMBT3904, Q12 MMBT3904, Q13 MMBT3906, U16 LM13700, U20 LM555, U3 TL074, U4 TL074

Commit message: big update, basic drum sequencing is working here
Parts:
- C14, C16: footprint Capacitor_SMD:C_0805_2012Metric_Pad1.15x1.40mm_HandSolder -> Capacitor_SMD:C_0603_1608Metric_Pad1.05x0.95mm_HandSolder
- R128, R129, R130, R131, R132, R133, R134, R135, R136, R137, R138, R139, R140, R141, R142, R143, R144, R145, R146, R147, R148, R149, R150, R151, R152, R153, R154, R155, R156, R157, R206: footprint Resistor_SMD:R_0805_2012Metric_Pad1.15x1.40mm_HandSolder -> Resistor_SMD:R_0603_1608Metric_Pad1.05x0.95mm_HandSolder
- R181, R182: footprint Capacitor_SMD:C_0805_2012Metric_Pad1.15x1.40mm_HandSolder -> Resistor_SMD:R_0603_1608Metric_Pad1.05x0.95mm_HandSolder
