File: harware_design/DrumMachineControlBoard/JackPanel.sch (KiCad schematic (older format))
At the start: 42 parts, among them J100 CYNB2-1, J103 CYNB3-1, J112 CYNB4-1, J128 CYNB5-1, J129 CYNB6-1, J130 CYNB1-W3, J131 CYNB2-W3, J132 CYNB3-W3, J141 CYNB4-W3, J143 CYNB5-W3, J144 CYNB6-W3, J74 Barrel_Jack, J75 MIX_LINE, J76 MIX_HEADPHONE, J79 Conn_01x03_Male, J80 CYNA1-1, J81 CYNA2-1, J82 CYNA3-1, J85 CYNA4-1, J86 CYNA5-1, J87 CYNA6-1, J88 CYNA1-W3, J89 CYNA2-W3, J90 CYNA3-W3, J91 CYNA4-W3, J97 CYNA5-W3, J98 CYNA6-W3, J99 CYNB1-1, U33 TL072

Commit message: big update, basic drum sequencing is working here
Parts:
- removed RV53: 10k, Potentiometer_THT:Potentiometer_Runtron_RM-065_Vertical, symbol Device:R_POT_TRIM_US
- removed U33: TL072, Package_SO:SOIC-8_3.9x4.9mm_P1.27mm, symbol Amplifier_Operational:TL072
- added C34, C35: 1u, Capacitor_SMD:CP_Elec_4x4.5, symbol Device:CP1_Small
- added C38, C39: 10u, Capacitor_SMD:CP_Elec_5x5.3, symbol Device:CP1_Small
- added C65, C66: 47n, Capacitor_SMD:C_0603_1608Metric_Pad1.05x0.95mm_HandSolder, symbol Device:C_Small
- added C67, C68: 220u, Capacitor_THT:CP_Radial_D5.0mm_P2.0mm_Bigger_Holes, symbol Device:CP1_Small
- added R183: 470k, Resistor_SMD:R_0603_1608Metric_Pad1.05x0.95mm_HandSolder, symbol Device:R_US
- added R184: 20k, Resistor_SMD:R_0603_1608Metric_Pad1.05x0.95mm_HandSolder, symbol Device:R_US
- added R185, R201: 10k, Resistor_SMD:R_0603_1608Metric_Pad1.05x0.95mm_HandSolder, symbol Device:R_US
- added R202, R203: 10, Resistor_SMD:R_0603_1608Metric_Pad1.05x0.95mm_HandSolder, symbol Device:R_US
- added RV53: 100k, mason_parts:masonsPotentiometer_Alpha_RD901F-40-00D_Single_Vertical, symbol Device:R_POT_US
- added U33, U34: LM386, Package_DIP:DIP-8_W7.62mm_Socket, symbol Amplifier_Audio:LM386
Connections:
- net +12V: now also U33.6 (V+), U34.6 (V+)
- net Earth: now also C38.2, C39.2, R184.1, R185.2, R201.2, R202.2, R203.2, RV53.3, U33.2 (-), U33.4 (GND), U34.2 (-), U34.4 (GND)
- net LINE_OUT: now also RV53.1
- net at J76.R1: now also C68.2
- net at J76.T1: now also C67.2
- new net: R183.2, RV53.2
- new net: C34.2, C35.2, R183.1, R184.2
- new net: C35.1, R201.1, U34.3 (+)
- new net: C66.1, C68.1, U34.5
- new net: C39.1, U34.7 (BYPASS)
- new net: C66.2, R203.1
- new net: C34.1, R185.1, U33.3 (+)
- new net: C65.1, C67.1, U33.5
- new net: C38.1, U33.7 (BYPASS)
- new net: C65.2, R202.1
- no-connect marks 5 -> 9
Other:
- moved on the sheet: J76A
