File: harware_design/DrumMachineControlBoard/LCD.sch (KiCad schematic (older format))
At the start: 3 parts, among them J145 Conn_01x08_Female, U24 Nokia5110

Commit message: big update, basic drum sequencing is working here
Parts:
- R177: footprint Resistor_SMD:R_0805_2012Metric_Pad1.15x1.40mm_HandSolder -> Resistor_SMD:R_0603_1608Metric_Pad1.05x0.95mm_HandSolder
Changed lines of the file:
@@
 F 0 "R177" H 3500 2250 50  0000 L CNN
 F 1 "220" H 3450 2150 50  0000 L CNN
-F 2 "Resistor_SMD:R_0805_2012Metric_Pad1.15x1.40mm_HandSolder" V 3690 2240 50  0001 C CNN
+F 2 "Resistor_SMD:R_0603_1608Metric_Pad1.05x0.95mm_HandSolder" V 3690 2240 50  0001 C CNN
 F 3 "~" H 3650 2250 50  0001 C CNN
 	1    3650 2250
