File: harware_design/DrumMachineControlBoard/LED Drivers.sch (KiCad schematic (older format))
At the start: 45 parts, among them J55 SR_AUX_1, J56 SR_AUX_2, J58 SR_AUX_3, J60 SR_AUX_4, U23 74HC595, U6 74HC595, U7 74HC595, U8 74HC595, U9 74HC595

Commit message: big update, basic drum sequencing is working here
Parts:
- R1, R10, R11, R12, R13, R14, R15, R16, R17, R18, R19, R2, R20, R21, R22, R23, R24, R25, R26, R27, R28, R29, R3, R30, R31, R32, R4, R5, R6, R7, R8, R9: footprint Resistor_SMD:R_0805_2012Metric_Pad1.15x1.40mm_HandSolder -> Resistor_SMD:R_0603_1608Metric_Pad1.05x0.95mm_HandSolder
