File: harware_design/DrumMachineControlBoard/MIDI.sch (KiCad schematic (older format))
At the start: 11 parts, among them J11 MIDI IN, J12 MIDI THRU, J13 MIDI OUT, U21 74LS04, U22 PC817

Commit message: big update, basic drum sequencing is working here
Parts:
- added R204: 220, Resistor_SMD:R_0603_1608Metric_Pad1.05x0.95mm_HandSolder, symbol Device:R_US
- R158, R159, R160, R161, R162: footprint Resistor_SMD:R_0805_2012Metric_Pad1.15x1.40mm_HandSolder -> Resistor_SMD:R_0603_1608Metric_Pad1.05x0.95mm_HandSolder
Connections:
- net +5V: now also R204.2
- net at J12.4: now also R204.1
- no-connect marks 13 -> 12
Changed lines of the file:
@@
 F 0 "R160" V 2145 1150 50  0000 C CNN
 F 1 "220" V 2236 1150 50  0000 C CNN
-F 2 "Resistor_SMD:R_0805_2012Metric_Pad1.15x1.40mm_HandSolder" V 2390 1140 50  0001 C CNN
+F 2 "Resistor_SMD:R_0603_1608Metric_Pad1.05x0.95mm_HandSolder" V 2390 1140 50  0001 C CNN
 F 3 "~" H 2350 1150 50  0001 C CNN
 	1    2350 1150
@@
 F 0 "R159" V 1995 4150 50  0000 C CNN
 F 1 "220" V 2086 4150 50  0000 C CNN
-F 2 "Resistor_SMD:R_0805_2012Metric_Pad1.15x1.40mm_HandSolder" V 2240 4140 50  0001 C CNN
+F 2 "Resistor_SMD:R_0603_1608Metric_Pad1.05x0.95mm_HandSolder" V 2240 4140 50  0001 C CNN
 F 3 "~" H 2200 4150 50  0001 C CNN
 	1    2200 4150
@@
 F 0 "R158" V 1695 4650 50  0000 C CNN
 F 1 "220" V 1786 4650 50  0000 C CNN
-F 2 "Resistor_SMD:R_0805_2012Metric_Pad1.15x1.40mm_HandSolder" V 1940 4640 50  0001 C CNN
+F 2 "Resistor_SMD:R_0603_1608Metric_Pad1.05x0.95mm_HandSolder" V 1940 4640 50  0001 C CNN
 F 3 "~" H 1900 4650 50  0001 C CNN
 	1    1900 4650
@@
 F 0 "R162" H 3782 904 50  0000 R CNN
 F 1 "1k" H 3782 995 50  0000 R CNN
-F 2 "Resistor_SMD:R_0805_2012Metric_Pad1.15x1.40mm_HandSolder" V 3890 940 50  0001 C CNN
+F 2 "Resistor_SMD:R_0603_1608Metric_Pad1.05x0.95mm_HandSolder" V 3890 940 50  0001 C CNN
 F 3 "~" H 3850 950 50  0001 C CNN
 	1    3850 950
@@
 F 0 "R161" V 2145 3100 50  0000 C CNN
 F 1 "220" V 2236 3100 50  0000 C CNN
-F 2 "Resistor_SMD:R_0805_2012Metric_Pad1.15x1.40mm_HandSolder" V 2390 3090 50  0001 C CNN
+F 2 "Resistor_SMD:R_0603_1608Metric_Pad1.05x0.95mm_HandSolder" V 2390 3090 50  0001 C CNN
 F 3 "~" H 2350 3100 50  0001 C CNN
 	1    2350 3100
@@
 NoConn ~ -2950 -2400
 NoConn ~ 350  -850
-NoConn ~ 1900 2550
 $Comp
 L Isolator:PC817 U22
@@
 Wire Wire Line
 	1900 4150 2050 4150
+$Comp
+L Device:R_US R204
+U 1 1 63831604
+P 2050 2350
+F 0 "R204" V 1845 2350 50  0000 C CNN
+F 1 "220" V 1936 2350 50  0000 C CNN
+F 2 "Resistor_SMD:R_0603_1608Metric_Pad1.05x0.95mm_HandSolder" V 2090 2340 50  0001 C CNN
+F 3 "~" H 2050 2350 50  0001 C CNN
+	1    2050 2350
+	-1   0    0    1
+$EndComp
+Wire Wire Line
+	2050 2500 2050 2550
+Wire Wire Line
+	2050 2550 1900 2550
+$Comp
+L power:+5V #PWR024
+U 1 1 63832540
+P 2050 2200
+F 0 "#PWR024" H 2050 2050 50  0001 C CNN
+F 1 "+5V" H 2065 2373 50  0000 C CNN
+F 2 "" H 2050 2200 50  0001 C CNN
+F 3 "" H 2050 2200 50  0001 C CNN
+	1    2050 2200
+	1    0    0    -1
+$EndComp
 $EndSCHEMATC
