File: harware_design/DrumMachineControlBoard/Noise.sch (KiCad schematic (older format))
At the start: 18 parts, among them J14 BD_Noise, J15 Snare_Noise, Q23 2N3904, U29 TL074

Commit message: big update, basic drum sequencing is working here
Parts:
- C36: footprint Capacitor_SMD:C_0805_2012Metric_Pad1.15x1.40mm_HandSolder -> Capacitor_SMD:C_0603_1608Metric_Pad1.05x0.95mm_HandSolder
- C37: footprint Capacitor_SMD:CP_Elec_4x4.5 -> Capacitor_SMD:CP_Elec_5x5.3
- R194, R195, R196, R197, R198: footprint Resistor_SMD:R_0805_2012Metric_Pad1.15x1.40mm_HandSolder -> Resistor_SMD:R_0603_1608Metric_Pad1.05x0.95mm_HandSolder
- R207, R208: footprint Capacitor_SMD:C_0805_2012Metric_Pad1.15x1.40mm_HandSolder -> Resistor_SMD:R_0603_1608Metric_Pad1.05x0.95mm_HandSolder
Changed lines of the file:
@@
 F 0 "R194" H 2268 3146 50  0000 L CNN
 F 1 "2M" H 2268 3055 50  0000 L CNN
-F 2 "Resistor_SMD:R_0805_2012Metric_Pad1.15x1.40mm_HandSolder" V 2240 3090 50  0001 C CNN
+F 2 "Resistor_SMD:R_0603_1608Metric_Pad1.05x0.95mm_HandSolder" V 2240 3090 50  0001 C CNN
 F 3 "~" H 2200 3100 50  0001 C CNN
 	1    2200 3100
@@
 F 0 "R196" V 2695 3800 50  0000 C CNN
 F 1 "4M7" V 2786 3800 50  0000 C CNN
-F 2 "Resistor_SMD:R_0805_2012Metric_Pad1.15x1.40mm_HandSolder" V 2940 3790 50  0001 C CNN
+F 2 "Resistor_SMD:R_0603_1608Metric_Pad1.05x0.95mm_HandSolder" V 2940 3790 50  0001 C CNN
 F 3 "~" H 2900 3800 50  0001 C CNN
 	1    2900 3800
@@
 F 0 "R195" H 2482 3954 50  0000 R CNN
 F 1 "100k" H 2482 4045 50  0000 R CNN
-F 2 "Resistor_SMD:R_0805_2012Metric_Pad1.15x1.40mm_HandSolder" V 2590 3990 50  0001 C CNN
+F 2 "Resistor_SMD:R_0603_1608Metric_Pad1.05x0.95mm_HandSolder" V 2590 3990 50  0001 C CNN
 F 3 "~" H 2550 4000 50  0001 C CNN
 	1    2550 4000
@@
 F 0 "C37" H 2641 4296 50  0000 L CNN
 F 1 "10u" H 2641 4205 50  0000 L CNN
-F 2 "Capacitor_SMD:CP_Elec_4x4.5" H 2550 4250 50  0001 C CNN
+F 2 "Capacitor_SMD:CP_Elec_5x5.3" H 2550 4250 50  0001 C CNN
 F 3 "~" H 2550 4250 50  0001 C CNN
 	1    2550 4250
@@
 F 0 "R197" V 4095 2800 50  0000 C CNN
 F 1 "10k" V 4186 2800 50  0000 C CNN
-F 2 "Resistor_SMD:R_0805_2012Metric_Pad1.15x1.40mm_HandSolder" V 4340 2790 50  0001 C CNN
+F 2 "Resistor_SMD:R_0603_1608Metric_Pad1.05x0.95mm_HandSolder" V 4340 2790 50  0001 C CNN
 F 3 "~" H 4300 2800 50  0001 C CNN
 	1    4300 2800
@@
 F 0 "R198" V 4095 3750 50  0000 C CNN
 F 1 "10k" V 4186 3750 50  0000 C CNN
-F 2 "Resistor_SMD:R_0805_2012Metric_Pad1.15x1.40mm_HandSolder" V 4340 3740 50  0001 C CNN
+F 2 "Resistor_SMD:R_0603_1608Metric_Pad1.05x0.95mm_HandSolder" V 4340 3740 50  0001 C CNN
 F 3 "~" H 4300 3750 50  0001 C CNN
 	1    4300 3750
@@
 F 0 "R208" H 1918 2396 50  0000 L CNN
 F 1 "470k" H 1918 2305 50  0000 L CNN
-F 2 "Capacitor_SMD:C_0805_2012Metric_Pad1.15x1.40mm_HandSolder" V 1890 2340 50  0001 C CNN
+F 2 "Resistor_SMD:R_0603_1608Metric_Pad1.05x0.95mm_HandSolder" V 1890 2340 50  0001 C CNN
 F 3 "~" H 1850 2350 50  0001 C CNN
 	1    1850 2350
@@
 F 0 "R207" V 1445 2150 50  0000 C CNN
 F 1 "470k" V 1536 2150 50  0000 C CNN
-F 2 "Capacitor_SMD:C_0805_2012Metric_Pad1.15x1.40mm_HandSolder" V 1690 2140 50  0001 C CNN
+F 2 "Resistor_SMD:R_0603_1608Metric_Pad1.05x0.95mm_HandSolder" V 1690 2140 50  0001 C CNN
 F 3 "~" H 1650 2150 50  0001 C CNN
 	1    1650 2150
@@
 F 0 "C36" V 2278 2900 50  0000 C CNN
 F 1 "100n" V 2187 2900 50  0000 C CNN
-F 2 "Capacitor_SMD:C_0805_2012Metric_Pad1.15x1.40mm_HandSolder" H 2050 2900 50  0001 C CNN
+F 2 "Capacitor_SMD:C_0603_1608Metric_Pad1.05x0.95mm_HandSolder" H 2050 2900 50  0001 C CNN
 F 3 "~" H 2050 2900 50  0001 C CNN
 	1    2050 2900
