File: harware_design/DrumMachineControlBoard/OutputMixer.sch (KiCad schematic (older format))
At the start: 79 parts, among them J118 Kick_Out, J119 Snare_Out, J120 CYN1_Out, J121 CYN2_Out, J122 Filt_Aux1, J123 Filt_Aux2, J2 Mix_Out, J21 DEL_SEND, J22 DEL_REC, J33 filter_CV, J40 mix_out, J53 Filter_IN, Q1 MMBT3906, Q2 Q_NPN_ECB, U16 LM13700, U17 SSI2144, U30 NE5532, U31 TL072, U32 TL072, U4 TL074

Commit message: big update, basic drum sequencing is working here
Parts:
- C10, C11, C12, C13, C9: footprint Capacitor_SMD:C_0805_2012Metric_Pad1.15x1.40mm_HandSolder -> Capacitor_SMD:C_0603_1608Metric_Pad1.05x0.95mm_HandSolder
- C5: footprint Capacitor_SMD:CP_Elec_6.3x7.7 -> Capacitor_SMD:CP_Elec_8x6.2
- C7, C8: footprint Capacitor_SMD:CP_Elec_4x4.5 -> Capacitor_SMD:CP_Elec_5x5.3
- R100, R101, R102, R103, R178, R179, R73, R74, R75, R76, R77, R78, R79, R80, R81, R82, R83, R84, R85, R86, R87, R88, R89, R90, R91, R92, R93, R94, R95, R96, R97, R98, R99: footprint Resistor_SMD:R_0805_2012Metric_Pad1.15x1.40mm_HandSolder -> Resistor_SMD:R_0603_1608Metric_Pad1.05x0.95mm_HandSolder
