File: harware_design/DrumMachineControlBoard/PWM Out.sch (KiCad schematic (older format))
At the start: 30 parts, among them J124 Kick_Vel, J125 Snare_Vel, J126 CYN1_Vel, J127 CYN2_Vel, U1 TL074, U2 TL072

Commit message: big update, basic drum sequencing is working here
Parts:
- C18, C19, C20, C21, C22, C23: footprint Capacitor_SMD:C_0805_2012Metric_Pad1.15x1.40mm_HandSolder -> Capacitor_SMD:C_0603_1608Metric_Pad1.05x0.95mm_HandSolder
- R163, R164, R165, R166, R167, R168, R169, R170, R171, R172, R173, R174: footprint Resistor_SMD:R_0805_2012Metric_Pad1.15x1.40mm_HandSolder -> Resistor_SMD:R_0603_1608Metric_Pad1.05x0.95mm_HandSolder
Changed lines of the file:
@@
 F 0 "R163" V 1995 1350 50  0000 C CNN
 F 1 "10k" V 2086 1350 50  0000 C CNN
-F 2 "Resistor_SMD:R_0805_2012Metric_Pad1.15x1.40mm_HandSolder" V 2240 1340 50  0001 C CNN
+F 2 "Resistor_SMD:R_0603_1608Metric_Pad1.05x0.95mm_HandSolder" V 2240 1340 50  0001 C CNN
 F 3 "~" H 2200 1350 50  0001 C CNN
 	1    2200 1350
@@
 F 0 "C18" H 2308 1454 50  0000 R CNN
 F 1 "100n" H 2308 1545 50  0000 R CNN
-F 2 "Capacitor_SMD:C_0805_2012Metric_Pad1.15x1.40mm_HandSolder" H 2400 1500 50  0001 C CNN
+F 2 "Capacitor_SMD:C_0603_1608Metric_Pad1.05x0.95mm_HandSolder" H 2400 1500 50  0001 C CNN
 F 3 "~" H 2400 1500 50  0001 C CNN
 	1    2400 1500
@@
 F 0 "R167" H 2632 2354 50  0000 R CNN
 F 1 "4k7" H 2632 2445 50  0000 R CNN
-F 2 "Resistor_SMD:R_0805_2012Metric_Pad1.15x1.40mm_HandSolder" V 2740 2390 50  0001 C CNN
+F 2 "Resistor_SMD:R_0603_1608Metric_Pad1.05x0.95mm_HandSolder" V 2740 2390 50  0001 C CNN
 F 3 "~" H 2700 2400 50  0001 C CNN
 	1    2700 2400
@@
 F 0 "C19" H 2308 3304 50  0000 R CNN
 F 1 "100n" H 2308 3395 50  0000 R CNN
-F 2 "Capacitor_SMD:C_0805_2012Metric_Pad1.15x1.40mm_HandSolder" H 2400 3350 50  0001 C CNN
+F 2 "Capacitor_SMD:C_0603_1608Metric_Pad1.05x0.95mm_HandSolder" H 2400 3350 50  0001 C CNN
 F 3 "~" H 2400 3350 50  0001 C CNN
 	1    2400 3350
@@
 F 0 "R164" V 1995 3200 50  0000 C CNN
 F 1 "10k" V 2086 3200 50  0000 C CNN
-F 2 "Resistor_SMD:R_0805_2012Metric_Pad1.15x1.40mm_HandSolder" V 2240 3190 50  0001 C CNN
+F 2 "Resistor_SMD:R_0603_1608Metric_Pad1.05x0.95mm_HandSolder" V 2240 3190 50  0001 C CNN
 F 3 "~" H 2200 3200 50  0001 C CNN
 	1    2200 3200
@@
 F 0 "R168" H 2682 3854 50  0000 R CNN
 F 1 "4k7" H 2682 3945 50  0000 R CNN
-F 2 "Resistor_SMD:R_0805_2012Metric_Pad1.15x1.40mm_HandSolder" V 2790 3890 50  0001 C CNN
+F 2 "Resistor_SMD:R_0603_1608Metric_Pad1.05x0.95mm_HandSolder" V 2790 3890 50  0001 C CNN
 F 3 "~" H 2750 3900 50  0001 C CNN
 	1    2750 3900
@@
 F 0 "C20" H 2358 4604 50  0000 R CNN
 F 1 "100n" H 2358 4695 50  0000 R CNN
-F 2 "Capacitor_SMD:C_0805_2012Metric_Pad1.15x1.40mm_HandSolder" H 2450 4650 50  0001 C CNN
+F 2 "Capacitor_SMD:C_0603_1608Metric_Pad1.05x0.95mm_HandSolder" H 2450 4650 50  0001 C CNN
 F 3 "~" H 2450 4650 50  0001 C CNN
 	1    2450 4650
@@
 F 0 "R165" V 2045 4500 50  0000 C CNN
 F 1 "10k" V 2136 4500 50  0000 C CNN
-F 2 "Resistor_SMD:R_0805_2012Metric_Pad1.15x1.40mm_HandSolder" V 2290 4490 50  0001 C CNN
+F 2 "Resistor_SMD:R_0603_1608Metric_Pad1.05x0.95mm_HandSolder" V 2290 4490 50  0001 C CNN
 F 3 "~" H 2250 4500 50  0001 C CNN
 	1    2250 4500
@@
 F 0 "R169" H 2732 5154 50  0000 R CNN
 F 1 "4k7" H 2732 5245 50  0000 R CNN
-F 2 "Resistor_SMD:R_0805_2012Metric_Pad1.15x1.40mm_HandSolder" V 2840 5190 50  0001 C CNN
+F 2 "Resistor_SMD:R_0603_1608Metric_Pad1.05x0.95mm_HandSolder" V 2840 5190 50  0001 C CNN
 F 3 "~" H 2800 5200 50  0001 C CNN
 	1    2800 5200
@@
 F 0 "C21" H 2358 5904 50  0000 R CNN
 F 1 "100n" H 2358 5995 50  0000 R CNN
-F 2 "Capacitor_SMD:C_0805_2012Metric_Pad1.15x1.40mm_HandSolder" H 2450 5950 50  0001 C CNN
+F 2 "Capacitor_SMD:C_0603_1608Metric_Pad1.05x0.95mm_HandSolder" H 2450 5950 50  0001 C CNN
 F 3 "~" H 2450 5950 50  0001 C CNN
 	1    2450 5950
@@
 F 0 "R166" V 2045 5800 50  0000 C CNN
 F 1 "10k" V 2136 5800 50  0000 C CNN
-F 2 "Resistor_SMD:R_0805_2012Metric_Pad1.15x1.40mm_HandSolder" V 2290 5790 50  0001 C CNN
+F 2 "Resistor_SMD:R_0603_1608Metric_Pad1.05x0.95mm_HandSolder" V 2290 5790 50  0001 C CNN
 F 3 "~" H 2250 5800 50  0001 C CNN
 	1    2250 5800
@@
 F 0 "R170" H 2732 6454 50  0000 R CNN
 F 1 "4k7" H 2732 6545 50  0000 R CNN
-F 2 "Resistor_SMD:R_0805_2012Metric_Pad1.15x1.40mm_HandSolder" V 2840 6490 50  0001 C CNN
+F 2 "Resistor_SMD:R_0603_1608Metric_Pad1.05x0.95mm_HandSolder" V 2840 6490 50  0001 C CNN
 F 3 "~" H 2800 6500 50  0001 C CNN
 	1    2800 6500
@@
 F 0 "R172" V 5745 1350 50  0000 C CNN
 F 1 "10k" V 5836 1350 50  0000 C CNN
-F 2 "Resistor_SMD:R_0805_2012Metric_Pad1.15x1.40mm_HandSolder" V 5990 1340 50  0001 C CNN
+F 2 "Resistor_SMD:R_0603_1608Metric_Pad1.05x0.95mm_HandSolder" V 5990 1340 50  0001 C CNN
 F 3 "~" H 5950 1350 50  0001 C CNN
 	1    5950 1350
@@
 F 0 "C23" H 6058 1454 50  0000 R CNN
 F 1 "100n" H 6058 1545 50  0000 R CNN
-F 2 "Capacitor_SMD:C_0805_2012Metric_Pad1.15x1.40mm_HandSolder" H 6150 1500 50  0001 C CNN
+F 2 "Capacitor_SMD:C_0603_1608Metric_Pad1.05x0.95mm_HandSolder" H 6150 1500 50  0001 C CNN
 F 3 "~" H 6150 1500 50  0001 C CNN
 	1    6150 1500
@@
 F 0 "R173" H 6382 2354 50  0000 R CNN
 F 1 "4k7" H 6382 2445 50  0000 R CNN
-F 2 "Resistor_SMD:R_0805_2012Metric_Pad1.15x1.40mm_HandSolder" V 6490 2390 50  0001 C CNN
+F 2 "Resistor_SMD:R_0603_1608Metric_Pad1.05x0.95mm_HandSolder" V 6490 2390 50  0001 C CNN
 F 3 "~" H 6450 2400 50  0001 C CNN
 	1    6450 2400
@@
 F 0 "C22" H 6008 3354 50  0000 R CNN
 F 1 "100n" H 6008 3445 50  0000 R CNN
-F 2 "Capacitor_SMD:C_0805_2012Metric_Pad1.15x1.40mm_HandSolder" H 6100 3400 50  0001 C CNN
+F 2 "Capacitor_SMD:C_0603_1608Metric_Pad1.05x0.95mm_HandSolder" H 6100 3400 50  0001 C CNN
 F 3 "~" H 6100 3400 50  0001 C CNN
 	1    6100 3400
@@
 F 0 "R174" H 6382 3904 50  0000 R CNN
 F 1 "4k7" H 6382 3995 50  0000 R CNN
-F 2 "Resistor_SMD:R_0805_2012Metric_Pad1.15x1.40mm_HandSolder" V 6490 3940 50  0001 C CNN
+F 2 "Resistor_SMD:R_0603_1608Metric_Pad1.05x0.95mm_HandSolder" V 6490 3940 50  0001 C CNN
 F 3 "~" H 6450 3950 50  0001 C CNN
 	1    6450 3950
@@
 F 0 "R171" V 5695 3250 50  0000 C CNN
 F 1 "10k" V 5786 3250 50  0000 C CNN
-F 2 "Resistor_SMD:R_0805_2012Metric_Pad1.15x1.40mm_HandSolder" V 5940 3240 50  0001 C CNN
+F 2 "Resistor_SMD:R_0603_1608Metric_Pad1.05x0.95mm_HandSolder" V 5940 3240 50  0001 C CNN
 F 3 "~" H 5900 3250 50  0001 C CNN
 	1    5900 3250
