File: harware_design/DrumMachineControlBoard/SpeakerAmp.sch (KiCad schematic (older format))
At the start: 7 parts, among them J16 spk_Conn, SW33 SW_SPDT, U28 NJM2073S

Commit message: big update, basic drum sequencing is working here
Parts:
- C24: footprint Capacitor_SMD:CP_Elec_4x4.5 -> Capacitor_SMD:CP_Elec_5x5.3
- C25: footprint Capacitor_SMD:C_0805_2012Metric_Pad1.15x1.40mm_HandSolder -> Capacitor_SMD:C_0603_1608Metric_Pad1.05x0.95mm_HandSolder
- R180: footprint Resistor_SMD:R_0805_2012Metric_Pad1.15x1.40mm_HandSolder -> Resistor_SMD:R_0603_1608Metric_Pad1.05x0.95mm_HandSolder
Changed lines of the file:
@@
 F 0 "C24" H 3691 1996 50  0000 L CNN
 F 1 "10u" H 3691 1905 50  0000 L CNN
-F 2 "Capacitor_SMD:CP_Elec_4x4.5" H 3600 1950 50  0001 C CNN
+F 2 "Capacitor_SMD:CP_Elec_5x5.3" H 3600 1950 50  0001 C CNN
 F 3 "~" H 3600 1950 50  0001 C CNN
 	1    3600 1950
@@
 F 0 "C25" H 3692 2646 50  0000 L CNN
 F 1 "100n" H 3692 2555 50  0000 L CNN
-F 2 "Capacitor_SMD:C_0805_2012Metric_Pad1.15x1.40mm_HandSolder" H 3600 2600 50  0001 C CNN
+F 2 "Capacitor_SMD:C_0603_1608Metric_Pad1.05x0.95mm_HandSolder" H 3600 2600 50  0001 C CNN
 F 3 "~" H 3600 2600 50  0001 C CNN
 	1    3600 2600
@@
 F 0 "R180" H 3132 1554 50  0000 R CNN
 F 1 "10k" H 3132 1645 50  0000 R CNN
-F 2 "Resistor_SMD:R_0805_2012Metric_Pad1.15x1.40mm_HandSolder" V 3240 1590 50  0001 C CNN
+F 2 "Resistor_SMD:R_0603_1608Metric_Pad1.05x0.95mm_HandSolder" V 3240 1590 50  0001 C CNN
 F 3 "~" H 3200 1600 50  0001 C CNN
 	1    3200 1600
