File: harware_design/DrumMachineControlBoard/TrigOuts.sch (KiCad schematic (older format))
At the start: 35 parts, among them J133 BD_TRIG_OUT, J134 SN_TRIG_OUT, J135 CYN1_TRIG_OUT, J136 CYN2_TRIG_OUT, J137 GLITCH_TRIG_OUT, J138 DIGI1_TRIG_OUT, J139 DIGI2_TRIG_OUT, J140 DIGI3_TRIG_OUT, J69 SR_AUX_6, J70 SR_AUX_5, Q15 2N7000, Q16 2N7000, Q17 2N7000, Q18 2N7000, Q19 2N7000, Q20 2N7000, Q21 2N7000, Q22 2N7000, U18 74HC595

Commit message: big update, basic drum sequencing is working here
Parts:
- R104, R105, R106, R107, R108, R109, R110, R111, R175, R176, R188, R189, R190, R191, R192, R193: footprint Capacitor_SMD:C_0805_2012Metric_Pad1.15x1.40mm_HandSolder -> Resistor_SMD:R_0603_1608Metric_Pad1.05x0.95mm_HandSolder
Changed lines of the file:
@@
 F 0 "R110" H 5068 946 50  0000 L CNN
 F 1 "2k2" H 5068 855 50  0000 L CNN
-F 2 "Capacitor_SMD:C_0805_2012Metric_Pad1.15x1.40mm_HandSolder" V 5040 890 50  0001 C CNN
+F 2 "Resistor_SMD:R_0603_1608Metric_Pad1.05x0.95mm_HandSolder" V 5040 890 50  0001 C CNN
 F 3 "~" H 5000 900 50  0001 C CNN
 	1    5000 900
@@
 F 0 "R104" V 4345 1250 50  0000 C CNN
 F 1 "470" V 4436 1250 50  0000 C CNN
-F 2 "Capacitor_SMD:C_0805_2012Metric_Pad1.15x1.40mm_HandSolder" V 4590 1240 50  0001 C CNN
+F 2 "Resistor_SMD:R_0603_1608Metric_Pad1.05x0.95mm_HandSolder" V 4590 1240 50  0001 C CNN
 F 3 "~" H 4550 1250 50  0001 C CNN
 	1    4550 1250
@@
 F 0 "R193" H 3618 6146 50  0000 L CNN
 F 1 "2k2" H 3618 6055 50  0000 L CNN
-F 2 "Capacitor_SMD:C_0805_2012Metric_Pad1.15x1.40mm_HandSolder" V 3590 6090 50  0001 C CNN
+F 2 "Resistor_SMD:R_0603_1608Metric_Pad1.05x0.95mm_HandSolder" V 3590 6090 50  0001 C CNN
 F 3 "~" H 3550 6100 50  0001 C CNN
 	1    3550 6100
@@
 F 0 "R191" V 2895 6450 50  0000 C CNN
 F 1 "470" V 2986 6450 50  0000 C CNN
-F 2 "Capacitor_SMD:C_0805_2012Metric_Pad1.15x1.40mm_HandSolder" V 3140 6440 50  0001 C CNN
+F 2 "Resistor_SMD:R_0603_1608Metric_Pad1.05x0.95mm_HandSolder" V 3140 6440 50  0001 C CNN
 F 3 "~" H 3100 6450 50  0001 C CNN
 	1    3100 6450
@@
 F 0 "R111" H 3518 2996 50  0000 L CNN
 F 1 "2k2" H 3518 2905 50  0000 L CNN
-F 2 "Capacitor_SMD:C_0805_2012Metric_Pad1.15x1.40mm_HandSolder" V 3490 2940 50  0001 C CNN
+F 2 "Resistor_SMD:R_0603_1608Metric_Pad1.05x0.95mm_HandSolder" V 3490 2940 50  0001 C CNN
 F 3 "~" H 3450 2950 50  0001 C CNN
 	1    3450 2950
@@
 F 0 "R105" V 2795 3300 50  0000 C CNN
 F 1 "470" V 2886 3300 50  0000 C CNN
-F 2 "Capacitor_SMD:C_0805_2012Metric_Pad1.15x1.40mm_HandSolder" V 3040 3290 50  0001 C CNN
+F 2 "Resistor_SMD:R_0603_1608Metric_Pad1.05x0.95mm_HandSolder" V 3040 3290 50  0001 C CNN
 F 3 "~" H 3000 3300 50  0001 C CNN
 	1    3000 3300
@@
 F 0 "R175" H 6568 2496 50  0000 L CNN
 F 1 "2k2" H 6568 2405 50  0000 L CNN
-F 2 "Capacitor_SMD:C_0805_2012Metric_Pad1.15x1.40mm_HandSolder" V 6540 2440 50  0001 C CNN
+F 2 "Resistor_SMD:R_0603_1608Metric_Pad1.05x0.95mm_HandSolder" V 6540 2440 50  0001 C CNN
 F 3 "~" H 6500 2450 50  0001 C CNN
 	1    6500 2450
@@
 F 0 "R106" V 5845 2800 50  0000 C CNN
 F 1 "470" V 5936 2800 50  0000 C CNN
-F 2 "Capacitor_SMD:C_0805_2012Metric_Pad1.15x1.40mm_HandSolder" V 6090 2790 50  0001 C CNN
+F 2 "Resistor_SMD:R_0603_1608Metric_Pad1.05x0.95mm_HandSolder" V 6090 2790 50  0001 C CNN
 F 3 "~" H 6050 2800 50  0001 C CNN
 	1    6050 2800
@@
 F 0 "R176" H 6568 3546 50  0000 L CNN
 F 1 "2k2" H 6568 3455 50  0000 L CNN
-F 2 "Capacitor_SMD:C_0805_2012Metric_Pad1.15x1.40mm_HandSolder" V 6540 3490 50  0001 C CNN
+F 2 "Resistor_SMD:R_0603_1608Metric_Pad1.05x0.95mm_HandSolder" V 6540 3490 50  0001 C CNN
 F 3 "~" H 6500 3500 50  0001 C CNN
 	1    6500 3500
@@
 F 0 "R107" V 5845 3850 50  0000 C CNN
 F 1 "470" V 5936 3850 50  0000 C CNN
-F 2 "Capacitor_SMD:C_0805_2012Metric_Pad1.15x1.40mm_HandSolder" V 6090 3840 50  0001 C CNN
+F 2 "Resistor_SMD:R_0603_1608Metric_Pad1.05x0.95mm_HandSolder" V 6090 3840 50  0001 C CNN
 F 3 "~" H 6050 3850 50  0001 C CNN
 	1    6050 3850
@@
 F 0 "R188" H 3618 5096 50  0000 L CNN
 F 1 "2k2" H 3618 5005 50  0000 L CNN
-F 2 "Capacitor_SMD:C_0805_2012Metric_Pad1.15x1.40mm_HandSolder" V 3590 5040 50  0001 C CNN
+F 2 "Resistor_SMD:R_0603_1608Metric_Pad1.05x0.95mm_HandSolder" V 3590 5040 50  0001 C CNN
 F 3 "~" H 3550 5050 50  0001 C CNN
 	1    3550 5050
@@
 F 0 "R108" V 2895 5400 50  0000 C CNN
 F 1 "470" V 2986 5400 50  0000 C CNN
-F 2 "Capacitor_SMD:C_0805_2012Metric_Pad1.15x1.40mm_HandSolder" V 3140 5390 50  0001 C CNN
+F 2 "Resistor_SMD:R_0603_1608Metric_Pad1.05x0.95mm_HandSolder" V 3140 5390 50  0001 C CNN
 F 3 "~" H 3100 5400 50  0001 C CNN
 	1    3100 5400
@@
 F 0 "R189" H 6018 6196 50  0000 L CNN
 F 1 "2k2" H 6018 6105 50  0000 L CNN
-F 2 "Capacitor_SMD:C_0805_2012Metric_Pad1.15x1.40mm_HandSolder" V 5990 6140 50  0001 C CNN
+F 2 "Resistor_SMD:R_0603_1608Metric_Pad1.05x0.95mm_HandSolder" V 5990 6140 50  0001 C CNN
 F 3 "~" H 5950 6150 50  0001 C CNN
 	1    5950 6150
@@
 F 0 "R109" V 5295 6500 50  0000 C CNN
 F 1 "470" V 5386 6500 50  0000 C CNN
-F 2 "Capacitor_SMD:C_0805_2012Metric_Pad1.15x1.40mm_HandSolder" V 5540 6490 50  0001 C CNN
+F 2 "Resistor_SMD:R_0603_1608Metric_Pad1.05x0.95mm_HandSolder" V 5540 6490 50  0001 C CNN
 F 3 "~" H 5500 6500 50  0001 C CNN
 	1    5500 6500
@@
 F 0 "R192" H 6018 5146 50  0000 L CNN
 F 1 "2k2" H 6018 5055 50  0000 L CNN
-F 2 "Capacitor_SMD:C_0805_2012Metric_Pad1.15x1.40mm_HandSolder" V 5990 5090 50  0001 C CNN
+F 2 "Resistor_SMD:R_0603_1608Metric_Pad1.05x0.95mm_HandSolder" V 5990 5090 50  0001 C CNN
 F 3 "~" H 5950 5100 50  0001 C CNN
 	1    5950 5100
@@
 F 0 "R190" V 5295 5450 50  0000 C CNN
 F 1 "470" V 5386 5450 50  0000 C CNN
-F 2 "Capacitor_SMD:C_0805_2012Metric_Pad1.15x1.40mm_HandSolder" V 5540 5440 50  0001 C CNN
+F 2 "Resistor_SMD:R_0603_1608Metric_Pad1.05x0.95mm_HandSolder" V 5540 5440 50  0001 C CNN
 F 3 "~" H 5500 5450 50  0001 C CNN
 	1    5500 5450
