File: harware_design/DrumMachineControlBoard/power_conns.sch (KiCad schematic (older format))
At the start: 6 parts, among them J47 PWR_CONN, J48 SNARE_PWR, J49 BD_PWR, J50 CYN1_PWR, J51 CYN2_PWR, J52 TWS_PWR

Commit message: big update, basic drum sequencing is working here
Changed lines of the file:
@@
 	0    1    1    0
 $EndComp
+$Comp
+L power:PWR_FLAG #FLG0101
+U 1 1 637FFCEE
+P 4250 2400
+F 0 "#FLG0101" H 4250 2475 50  0001 C CNN
+F 1 "PWR_FLAG" H 4250 2573 50  0000 C CNN
+F 2 "" H 4250 2400 50  0001 C CNN
+F 3 "~" H 4250 2400 50  0001 C CNN
+	1    4250 2400
+	1    0    0    -1
+$EndComp
+$Comp
+L power:Earth #PWR0220
+U 1 1 638002A7
+P 4250 2400
+F 0 "#PWR0220" H 4250 2150 50  0001 C CNN
+F 1 "Earth" H 4250 2250 50  0001 C CNN
+F 2 "" H 4250 2400 50  0001 C CNN
+F 3 "~" H 4250 2400 50  0001 C CNN
+	1    4250 2400
+	1    0    0    -1
+$EndComp
+$Comp
+L power:PWR_FLAG #FLG0102
+U 1 1 63806D4A
+P 4650 2400
+F 0 "#FLG0102" H 4650 2475 50  0001 C CNN
+F 1 "PWR_FLAG" H 4650 2573 50  0000 C CNN
+F 2 "" H 4650 2400 50  0001 C CNN
+F 3 "~" H 4650 2400 50  0001 C CNN
+	1    4650 2400
+	1    0    0    -1
+$EndComp
+$Comp
+L power:PWR_FLAG #FLG0103
+U 1 1 6380734A
+P 5050 2400
+F 0 "#FLG0103" H 5050 2475 50  0001 C CNN
+F 1 "PWR_FLAG" H 5050 2573 50  0000 C CNN
+F 2 "" H 5050 2400 50  0001 C CNN
+F 3 "~" H 5050 2400 50  0001 C CNN
+	1    5050 2400
+	1    0    0    -1
+$EndComp
+$Comp
+L power:PWR_FLAG #FLG0104
+U 1 1 63807581
+P 5450 2400
+F 0 "#FLG0104" H 5450 2475 50  0001 C CNN
+F 1 "PWR_FLAG" H 5450 2573 50  0000 C CNN
+F 2 "" H 5450 2400 50  0001 C CNN
+F 3 "~" H 5450 2400 50  0001 C CNN
+	1    5450 2400
+	1    0    0    -1
+$EndComp
+$Comp
+L power:+12V #PWR0221
+U 1 1 63807983
+P 4650 2400
+F 0 "#PWR0221" H 4650 2250 50  0001 C CNN
+F 1 "+12V" V 4665 2528 50  0000 L CNN
+F 2 "" H 4650 2400 50  0001 C CNN
+F 3 "" H 4650 2400 50  0001 C CNN
+	1    4650 2400
+	-1   0    0    1
+$EndComp
+$Comp
+L power:+5V #PWR0222
+U 1 1 6380814F
+P 5050 2400
+F 0 "#PWR0222" H 5050 2250 50  0001 C CNN
+F 1 "+5V" V 5065 2528 50  0000 L CNN
+F 2 "" H 5050 2400 50  0001 C CNN
+F 3 "" H 5050 2400 50  0001 C CNN
+	1    5050 2400
+	-1   0    0    1
+$EndComp
+$Comp
+L power:-12V #PWR0411
+U 1 1 6380888A
+P 5450 2400
+F 0 "#PWR0411" H 5450 2500 50  0001 C CNN
+F 1 "-12V" V 5465 2528 50  0000 L CNN
+F 2 "" H 5450 2400 50  0001 C CNN
+F 3 "" H 5450 2400 50  0001 C CNN
+	1    5450 2400
+	-1   0    0    1
+$EndComp
 $EndSCHEMATC
