File: harware_design/DrumMachineControlBoard/rotaryEncoders.sch (KiCad schematic (older format))
At the start: 14 parts, among them SW1 DataEnc, SW2 TempoEnc

Commit message: big update, basic drum sequencing is working here
Parts:
- C1, C2, C3, C4: footprint Capacitor_SMD:C_0805_2012Metric_Pad1.15x1.40mm_HandSolder -> Capacitor_SMD:C_0603_1608Metric_Pad1.05x0.95mm_HandSolder
- R33, R34, R35, R36, R37, R38, R39, R40: footprint Resistor_SMD:R_0805_2012Metric_Pad1.15x1.40mm_HandSolder -> Resistor_SMD:R_0603_1608Metric_Pad1.05x0.95mm_HandSolder
Changed lines of the file:
@@
 F 0 "R33" V 1245 2000 50  0000 C CNN
 F 1 "10k" V 1336 2000 50  0000 C CNN
-F 2 "Resistor_SMD:R_0805_2012Metric_Pad1.15x1.40mm_HandSolder" V 1490 1990 50  0001 C CNN
+F 2 "Resistor_SMD:R_0603_1608Metric_Pad1.05x0.95mm_HandSolder" V 1490 1990 50  0001 C CNN
 F 3 "~" H 1450 2000 50  0001 C CNN
 	1    1450 2000
@@
 F 0 "R36" V 2045 2000 50  0000 C CNN
 F 1 "10k" V 2136 2000 50  0000 C CNN
-F 2 "Resistor_SMD:R_0805_2012Metric_Pad1.15x1.40mm_HandSolder" V 2290 1990 50  0001 C CNN
+F 2 "Resistor_SMD:R_0603_1608Metric_Pad1.05x0.95mm_HandSolder" V 2290 1990 50  0001 C CNN
 F 3 "~" H 2250 2000 50  0001 C CNN
 	1    2250 2000
@@
 F 0 "R34" H 1582 2204 50  0000 R CNN
 F 1 "10k" H 1582 2295 50  0000 R CNN
-F 2 "Resistor_SMD:R_0805_2012Metric_Pad1.15x1.40mm_HandSolder" V 1690 2240 50  0001 C CNN
+F 2 "Resistor_SMD:R_0603_1608Metric_Pad1.05x0.95mm_HandSolder" V 1690 2240 50  0001 C CNN
 F 3 "~" H 1650 2250 50  0001 C CNN
 	1    1650 2250
@@
 F 0 "R35" H 1982 2204 50  0000 R CNN
 F 1 "10k" H 1982 2295 50  0000 R CNN
-F 2 "Resistor_SMD:R_0805_2012Metric_Pad1.15x1.40mm_HandSolder" V 2090 2240 50  0001 C CNN
+F 2 "Resistor_SMD:R_0603_1608Metric_Pad1.05x0.95mm_HandSolder" V 2090 2240 50  0001 C CNN
 F 3 "~" H 2050 2250 50  0001 C CNN
 	1    2050 2250
@@
 F 0 "C1" V 1579 2450 50  0000 C CNN
 F 1 "10n" V 1488 2450 50  0000 C CNN
-F 2 "Capacitor_SMD:C_0805_2012Metric_Pad1.15x1.40mm_HandSolder" H 1350 2450 50  0001 C CNN
+F 2 "Capacitor_SMD:C_0603_1608Metric_Pad1.05x0.95mm_HandSolder" H 1350 2450 50  0001 C CNN
 F 3 "~" H 1350 2450 50  0001 C CNN
 	1    1350 2450
@@
 F 0 "C2" V 2579 2450 50  0000 C CNN
 F 1 "10n" V 2488 2450 50  0000 C CNN
-F 2 "Capacitor_SMD:C_0805_2012Metric_Pad1.15x1.40mm_HandSolder" H 2350 2450 50  0001 C CNN
+F 2 "Capacitor_SMD:C_0603_1608Metric_Pad1.05x0.95mm_HandSolder" H 2350 2450 50  0001 C CNN
 F 3 "~" H 2350 2450 50  0001 C CNN
 	1    2350 2450
@@
 F 0 "R37" V 3045 2000 50  0000 C CNN
 F 1 "10k" V 3136 2000 50  0000 C CNN
-F 2 "Resistor_SMD:R_0805_2012Metric_Pad1.15x1.40mm_HandSolder" V 3290 1990 50  0001 C CNN
+F 2 "Resistor_SMD:R_0603_1608Metric_Pad1.05x0.95mm_HandSolder" V 3290 1990 50  0001 C CNN
 F 3 "~" H 3250 2000 50  0001 C CNN
 	1    3250 2000
@@
 F 0 "R40" V 3845 2000 50  0000 C CNN
 F 1 "10k" V 3936 2000 50  0000 C CNN
-F 2 "Resistor_SMD:R_0805_2012Metric_Pad1.15x1.40mm_HandSolder" V 4090 1990 50  0001 C CNN
+F 2 "Resistor_SMD:R_0603_1608Metric_Pad1.05x0.95mm_HandSolder" V 4090 1990 50  0001 C CNN
 F 3 "~" H 4050 2000 50  0001 C CNN
 	1    4050 2000
@@
 F 0 "R38" H 3382 2204 50  0000 R CNN
 F 1 "10k" H 3382 2295 50  0000 R CNN
-F 2 "Resistor_SMD:R_0805_2012Metric_Pad1.15x1.40mm_HandSolder" V 3490 2240 50  0001 C CNN
+F 2 "Resistor_SMD:R_0603_1608Metric_Pad1.05x0.95mm_HandSolder" V 3490 2240 50  0001 C CNN
 F 3 "~" H 3450 2250 50  0001 C CNN
 	1    3450 2250
@@
 F 0 "R39" H 3782 2204 50  0000 R CNN
 F 1 "10k" H 3782 2295 50  0000 R CNN
-F 2 "Resistor_SMD:R_0805_2012Metric_Pad1.15x1.40mm_HandSolder" V 3890 2240 50  0001 C CNN
+F 2 "Resistor_SMD:R_0603_1608Metric_Pad1.05x0.95mm_HandSolder" V 3890 2240 50  0001 C CNN
 F 3 "~" H 3850 2250 50  0001 C CNN
 	1    3850 2250
@@
 F 0 "C3" V 3379 2450 50  0000 C CNN
 F 1 "10n" V 3288 2450 50  0000 C CNN
-F 2 "Capacitor_SMD:C_0805_2012Metric_Pad1.15x1.40mm_HandSolder" H 3150 2450 50  0001 C CNN
+F 2 "Capacitor_SMD:C_0603_1608Metric_Pad1.05x0.95mm_HandSolder" H 3150 2450 50  0001 C CNN
 F 3 "~" H 3150 2450 50  0001 C CNN
 	1    3150 2450
@@
 F 0 "C4" V 4379 2450 50  0000 C CNN
 F 1 "10n" V 4288 2450 50  0000 C CNN
-F 2 "Capacitor_SMD:C_0805_2012Metric_Pad1.15x1.40mm_HandSolder" H 4150 2450 50  0001 C CNN
+F 2 "Capacitor_SMD:C_0603_1608Metric_Pad1.05x0.95mm_HandSolder" H 4150 2450 50  0001 C CNN
 F 3 "~" H 4150 2450 50  0001 C CNN
 	1    4150 2450
